File: breakout/breakout.brd (EAGLE design)
At the start: 505 x 160 mm, 244 parts, among them J17 1789074, J26 69168-124HLF, J29 SJ1-3514-SMT-TR, J31 69168-116HLF, J32 12226-8250-00FR, J33 1888276, J34 69168-116HLF, J35 1888276, Q1 SI1012R, Q2 SI1012R, Q3 SI1012R, Q4 SI1012R, Q5 SI1012R, Q6 SI1012R, Q7 SI1012R, Q8 SI1012R, Q9 IRFML8244TRPBF, U1 SK6805-E-J, U10 TXB0101, U11 SK6805-E-J, U12 SK6805-E-J, U13 SK6805-E-J, U14 SK6805-E-J, U15 SK6805-E-J, U16 SK6805-E-J, U17 SK6805-E-J, U18 SK6805-E-J, U19 SK6805-E-J, U2 SK6805-E-J, U20 SK6805-E-J, U21 SK6805-E-J, U22 SK6805-E-J, U23 SK6805-E-J, U24 SK6805-E-J, U25 SK6805-E-J, U26 SK6805-E-J, U27 SK6805-E-J, U28 SK6805-E-J, U29 SK6805-E-J, U3 SK6805-E-J, U30 SK6805-E-J, U31 SK6805-E-J, U32 SK6805-E-J, U33 SK6805-E-J, U34 SK6805-E-J, U35 SK6805-E-J, U36 SK6805-E-J, U37 SK6805-E-J, U38 SK6805-E-J, U39 SK6805-E-J, U4 SK6805-E-J, U40 SK6805-E-J, U41 SK6805-E-J, U42 SK6805-E-J, U43 G6K-2F-RF, U44 G6K-2F-RF, U45 G6K-2F-RF, U46 G6K-2F-RF, U47 LTM4622A, U48 SI8610, U49 TINY-FPGA-BX, U5 SK6805-E-J, U50 TCA9555, U51 FIN1032MTCX, U52 SN65LVDS9638DGN, U53 SN65LVDS9638DGN, U6 SK6805-E-J, U7 SK6805-E-J, U8 SK6805-E-J, U9 SK6805-E-J

Commit message: Add .gitignore
- Update schematic part numbers to match BOM
Parts:
- R25: value 100 -> 4.7k
- R27: value 270, 0.5W -> 100; device jonnew:0805 -> jonnew:0402
- R43: value 4.7k -> 270, 0.5W; device jonnew:0402 -> jonnew:0805
- moved C42 59.5 mm to (439.4, 74.9), turned to 0 degrees
- moved C43 59.5 mm to (480.4, 118.0), turned to 270 degrees
- moved R42 48.0 mm to (480.1, 126.3)
- moved R41 47.5 mm to (432.9, 121.4)
- moved R40 43.9 mm to (476.5, 126.3)
- moved R39 43.6 mm to (432.9, 125.4)
- moved R37 40.1 mm to (432.9, 129.4)
- moved R38 40.0 mm to (472.9, 126.3)
- moved R36 36.5 mm to (469.3, 126.3)
- moved R35 29.8 mm to (440.9, 117.4)
- moved R43 26.6 mm to (432.9, 117.4)
- moved R34 26.3 mm to (465.7, 126.3)
- moved R33 25.3 mm to (440.9, 121.4)
- moved R25 22.9 mm to (450.8, 97.7), turned to 180 degrees
- moved R32 21.8 mm to (462.1, 126.3)
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Connections:
- net +12V: now also R25.2; no longer R43.2
- net +3V3: now also C42.2; no longer C43.2
- net +5V0: now also C43.2; no longer C42.2
- net +5V0_GOOD: now also R25.1; no longer R43.1
- net DIN0: now also R43.2; no longer R42.2
- net DIN0_P: now also R43.1; no longer R42.1
- net DIN1: now also R35.2; no longer R34.2
- net DIN1_P: now also R35.1; no longer R34.1
- net DIN2: now also R41.2; no longer R40.2
- net DIN2_P: now also R41.1; no longer R40.1
- net DIN3: now also R33.2; no longer R32.2
- net DIN3_P: now also R33.1; no longer R32.1
- net DIN4: now also R39.2; no longer R38.2
- net DIN4_P: now also R39.1; no longer R38.1
- net DIN5: now also R31.2; no longer R30.2
- net DIN5_P: now also R31.1; no longer R30.1
- net DIN6: now also R37.2; no longer R36.2
- net DIN6_P: now also R37.1; no longer R36.1
- net DIN7: now also R29.2; no longer R28.2
- net DIN7_P: now also R29.1; no longer R28.1
- net DOUT0: now also R28.2; no longer R27.2
- net DOUT0_P: now also R28.1; no longer R27.1
- net DOUT1: now also R30.2; no longer R29.2
- net DOUT1_P: now also R30.1; no longer R29.1
- net DOUT2: now also R32.2; no longer R31.2
- net DOUT2_P: now also R32.1; no longer R31.1
- net DOUT3: now also R34.2; no longer R33.2
- net DOUT3_P: now also R34.1; no longer R33.1
- net DOUT4: now also R36.2; no longer R35.2
- net DOUT4_P: now also R36.1; no longer R35.1
- net DOUT5: now also R38.2; no longer R37.2
- net DOUT5_P: now also R38.1; no longer R37.1
- net DOUT6: now also R40.2; no longer R39.2
- net DOUT6_P: now also R40.1; no longer R39.1
- net DOUT7: now also R42.2; no longer R41.2
- net DOUT7_P: now also R42.1; no longer R41.1
- net LVDS_DOUT0_N: now also R26.1; no longer R25.1
- net LVDS_DOUT0_P: now also R26.2; no longer R25.2
- net LVDS_DOUT1_N: now also R27.1; no longer R26.1
- net LVDS_DOUT1_P: now also R27.2; no longer R26.2
