File: breakout/breakout.brd (EAGLE design)
At the start: 505 x 160 mm, 244 parts, among them J17 1789074, J26 69168-124HLF, J29 SJ1-3514-SMT-TR, J31 69168-116HLF, J32 12226-8250-00FR, J33 1888276, J34 69168-116HLF, J35 1888276, Q1 SI1012R, Q2 SI1012R, Q3 SI1012R, Q4 SI1012R, Q5 SI1012R, Q6 SI1012R, Q7 SI1012R, Q8 SI1012R, Q9 IRFML8244TRPBF, U1 SK6805-E-J, U10 TXB0101, U11 SK6805-E-J, U12 SK6805-E-J, U13 SK6805-E-J, U14 SK6805-E-J, U15 SK6805-E-J, U16 SK6805-E-J, U17 SK6805-E-J, U18 SK6805-E-J, U19 SK6805-E-J, U2 SK6805-E-J, U20 SK6805-E-J, U21 SK6805-E-J, U22 SK6805-E-J, U23 SK6805-E-J, U24 SK6805-E-J, U25 SK6805-E-J, U26 SK6805-E-J, U27 SK6805-E-J, U28 SK6805-E-J, U29 SK6805-E-J, U3 SK6805-E-J, U30 SK6805-E-J, U31 SK6805-E-J, U32 SK6805-E-J, U33 SK6805-E-J, U34 SK6805-E-J, U35 SK6805-E-J, U36 SK6805-E-J, U37 SK6805-E-J, U38 SK6805-E-J, U39 SK6805-E-J, U4 SK6805-E-J, U40 SK6805-E-J, U41 SK6805-E-J, U42 SK6805-E-J, U43 G6K-2F-RF, U44 G6K-2F-RF, U45 G6K-2F-RF, U46 G6K-2F-RF, U47 LTM4622A, U48 SI8610, U49 TINY-FPGA-BX, U5 SK6805-E-J, U50 TCA9555, U51 FIN1032MTCX, U52 SN65LVDS9638DGN, U53 SN65LVDS9638DGN, U6 SK6805-E-J, U7 SK6805-E-J, U8 SK6805-E-J, U9 SK6805-E-J

Commit message: Updated the schematic to use Harp timestamp bus as input.
The layout (.brd) is not ready yet.

Replaced U48 SI8610 with U48 TLV70033DDCR (adds  extra BOM line. PN TLV70033DDCR)
Replaced C41 0402 0.1uF with C41 0805 10uF (same PN as C40 to not add extra BOM line)
Replaced C43 0402 0.1uF with C43 0805 10uF (same PN as C40 to not add extra BOM line)
Added R44 0402 13.3k (same PN as R19 to not add extra BOM line)
Added R45 0402 10R (adds extra BOM line. PN CRCW040210R0FKEDHP)

New BOM lines: 2
Replaced components: 3
Parts:
- added R44: 13.3k, jonnew:0402
- added R45: 10R, jonnew:0402
- C41, C43: value 0.1uF -> 10uF; device jonnew:0402 -> jonnew:0805
- U48: value SI8610 -> TLV70033DDCR; device CNP-ics 2:SO-08 -> harp input expander:TSOT23-5
- moved C43 516.6 mm to (-15.6, -26.3), turned to 0 degrees
- moved U48 506.0 mm to (-16.3, -4.10), turned to 0 degrees
- moved C41 504.5 mm to (-15.6, -20.7), turned to 0 degrees
Connections:
- removed net HARP_CLKOUT: U48.2, U49.24
- removed net N$17: C41.2, J29.5, U48.5
- removed net N$18: J29.4, U48.6
- new net HARP_CLKIN: J29.4, R44.2, U49.24
- new net N$85: C43.1, R45.1, U48.5
- net +5V0: now also C41.1, U48.3; no longer C43.2
- net GND: now also C41.2, C43.2, J29.5, U48.2; no longer C43.1, U48.4
- net N$16: now also R44.1, R45.2; no longer C41.1, U48.8
Routing:
- net N$17: track 20.7 -> 0.00 mm, vias 2 -> 0
- net HARP_CLKIN: track 0.00 -> 15.0 mm, vias 0 -> 3
- net N$18: track 12.6 -> 0.00 mm, vias 2 -> 0
- net GND: track 33.3 -> 44.5 mm, vias 1159 -> 1160
- net HARP_CLKOUT: track 5.87 -> 0.00 mm, vias 1 -> 0
- net +5V0: track 1328.5 -> 1323.8 mm
- net N$16: track 23.3 -> 19.8 mm

Commit message: Updated the layout to use Harp timestamp bus as input.
Parts:
- moved C41 516.3 mm to (481.7, 118.1), turned to 270 degrees
- moved C43 511.9 mm to (475.5, 118.1), turned to 90 degrees
- moved R45 511.9 mm to (471.5, 118.8), turned to 180 degrees
- moved U48 509.8 mm to (478.6, 118.1), turned to 180 degrees
- moved R44 509.7 mm to (471.5, 116.0)
Routing:
- net GND: track 44.5 -> 28.8 mm, vias 1160 -> 1164
- net +5V0: track 1323.8 -> 1335.9 mm, vias 59 -> 60
- net N$85: track 0.00 -> 11.7 mm
- net HARP_CLKIN: track 15.0 -> 11.8 mm, vias 3 -> 2
- net N$16: track 19.8 -> 23.0 mm
