File: breakout/breakout.brd (EAGLE design)
At the start: 505 x 160 mm, 246 parts, among them J17 1789074, J26 69168-124HLF, J29 SJ1-3514-SMT-TR, J31 69168-116HLF, J32 12226-8250-00FR, J33 1888276, J34 69168-116HLF, J35 1888276, Q1 SI1012R, Q2 SI1012R, Q3 SI1012R, Q4 SI1012R, Q5 SI1012R, Q6 SI1012R, Q7 SI1012R, Q8 SI1012R, Q9 IRFML8244TRPBF, U1 SK6805-E-J, U10 TXB0101, U11 SK6805-E-J, U12 SK6805-E-J, U13 SK6805-E-J, U14 SK6805-E-J, U15 SK6805-E-J, U16 SK6805-E-J, U17 SK6805-E-J, U18 SK6805-E-J, U19 SK6805-E-J, U2 SK6805-E-J, U20 SK6805-E-J, U21 SK6805-E-J, U22 SK6805-E-J, U23 SK6805-E-J, U24 SK6805-E-J, U25 SK6805-E-J, U26 SK6805-E-J, U27 SK6805-E-J, U28 SK6805-E-J, U29 SK6805-E-J, U3 SK6805-E-J, U30 SK6805-E-J, U31 SK6805-E-J, U32 SK6805-E-J, U33 SK6805-E-J, U34 SK6805-E-J, U35 SK6805-E-J, U36 SK6805-E-J, U37 SK6805-E-J, U38 SK6805-E-J, U39 SK6805-E-J, U4 SK6805-E-J, U40 SK6805-E-J, U41 SK6805-E-J, U42 SK6805-E-J, U43 G6K-2F-RF, U44 G6K-2F-RF, U45 G6K-2F-RF, U46 G6K-2F-RF, U47 LTM4622A, U48 TLV70033DDCR, U49 TINY-FPGA-BX, U5 SK6805-E-J, U50 TCA9555, U51 FIN1032MTCX, U52 SN65LVDS9638DGN, U53 SN65LVDS9638DGN, U6 SK6805-E-J, U7 SK6805-E-J, U8 SK6805-E-J, U9 SK6805-E-J

Commit message: Updated BOM to PN available in the market.
U48 - PN TLV70033DDCR changed to LP5951MFX-3.3/NOPB
R45 - PN CRCW040210R0FKEDHP changed to ERJ-PA2J100X
Parts:
- U48: value TLV70033DDCR -> LP5951MFX-3.3/NOPB
Changed lines of the file:
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@@
 <attribute name="NAME" x="452.157" y="97.162" size="1.016" layer="25" font="vector" ratio="18"/>
 </element>
-<element name="U48" library="harp input expander" package="TSOT23-5" value="TLV70033DDCR" x="478.6" y="118.1" smashed="yes" rot="R180">
+<element name="U48" library="harp input expander" package="TSOT23-5" value="LP5951MFX-3.3/NOPB" x="478.6" y="118.1" smashed="yes" rot="R180">
 <attribute name="MPN" value="TLV70033DDCR" x="485" y="124.8" size="1.778" layer="27" rot="R180" display="off"/>
 <attribute name="NAME" x="479.797" y="115.736" size="1.016" layer="25" font="vector" ratio="18" rot="R180"/>

Commit message: Changed separation method to mouse bites.
The design of the functional circuitry of the PCB has no difference
The previous commit can be used for production, it's the same board's revision.
Other:
- board size 505 x 160 mm -> 485 x 160 mm
- board text removed: "V-CUT"
